File: electronics/panel-board/power.kicad_sch (KiCad schematic)
At the start: 23 parts, among them J18 Barrel_Jack_MountingPin, U12 AMS1117-3.3, U13 TPS5430DDA

Commit message: Update PadBUS standard
Parts:
- TP17: value (none) -> TestPoint; footprint (none) -> TestPoint:TestPoint_Pad_D2.0mm
Changed lines of the file:
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@@
       (effects (font (size 1.27 1.27)) (justify left))
     )
-    (property "Value" "" (id 1) (at 167.767 40.3102 0)
+    (property "Value" "TestPoint" (id 1) (at 167.767 40.3102 0)
       (effects (font (size 1.27 1.27)) (justify left) hide)
     )
-    (property "Footprint" "" (id 2) (at 171.45 41.91 0)
+    (property "Footprint" "TestPoint:TestPoint_Pad_D2.0mm" (id 2) (at 171.45 41.91 0)
       (effects (font (size 1.27 1.27)) hide)
     )
