File: electronics/panel-board/controller.kicad_sch (KiCad schematic)
At the start: 18 parts, among them U9 STM32G431CBT6, Y1 8MHz

Commit message: Update PadBUS standard
Connections:
- net NODE_EN_L: now reaches U9.30 (PA8)
- net NODE_EN_R: now reaches U9.31 (PA9)
- no-connect marks 9 -> 7
Changed lines of the file:
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@@
   (no_connect (at 173.99 71.12))
   (no_connect (at 173.99 68.58))
-  (no_connect (at 120.65 101.6))
-  (no_connect (at 120.65 104.14))
   (no_connect (at 120.65 106.68))
   (no_connect (at 120.65 76.2))
@@
     (stroke (width 0) (type default) (color 0 0 0 0))
   )
+  (wire (pts (xy 118.11 104.14) (xy 120.65 104.14))
+    (stroke (width 0) (type default) (color 0 0 0 0))
+  )
   (wire (pts (xy 119.38 54.61) (xy 119.38 58.42))
     (stroke (width 0) (type default) (color 0 0 0 0))
@@
   )
   (wire (pts (xy 113.03 121.92) (xy 113.03 124.46))
+    (stroke (width 0) (type default) (color 0 0 0 0))
+  )
+  (wire (pts (xy 118.11 101.6) (xy 120.65 101.6))
     (stroke (width 0) (type default) (color 0 0 0 0))
   )
@@
     (effects (font (size 1.27 1.27)) (justify right))
   )
+  (hierarchical_label "NODE_EN_L" (shape bidirectional) (at 118.11 101.6 180)
+    (effects (font (size 1.27 1.27)) (justify right))
+  )
   (hierarchical_label "CAN_TX" (shape output) (at 176.53 81.28 0)
     (effects (font (size 1.27 1.27)) (justify left))
@@
     (effects (font (size 1.27 1.27)) (justify left))
   )
+  (hierarchical_label "NODE_EN_R" (shape bidirectional) (at 118.11 104.14 180)
+    (effects (font (size 1.27 1.27)) (justify right))
+  )
   (hierarchical_label "LED_SEG_UL" (shape output) (at 176.53 88.9 0)

Commit message: Prelim schematic for FSR+LC gain/adj dig control
Connections:
- net LC_ADJ_DPOT_EN: now reaches U9.32 (PA10)
- net FSR_ADJ_DPOT_EN: now reaches U9.39 (PA15)
- net DPOT_DATA: now reaches U9.41 (PB4)
- net DPOT_CLK: now reaches U9.42 (PB5)
- net LC_GAIN_DPOT_EN: now reaches U9.43 (PB6)
- net FSR_GAIN_DPOT_EN: now reaches U9.44 (PB7)
- no-connect marks 7 -> 1
Other:
- moved on the sheet: C29, C30, R33, Y1
